Commit message: fix2

File: src/description/urdf/robot.urdf.xacro (robot description, xacro)
@@ -1,16 +1,49 @@
 <?xml version="1.0"?>
-<robot xmlns:xacro="http://www.ros.org/wiki/xacro"  name="call_robot">
-    <xacro:arg name="use_ros2_control" default="true"/>
-    <xacro:arg name="robot_name" default="Minibot"/>
-    <xacro:include filename="robot_core.xacro">
-        <xacro:arg name="robot_name" value="$(arg robot_name)"/>
-    </xacro:include>
-    <xacro:unless value="$(arg use_ros2_control)">
-        <xacro:include filename="gazebo_control.xacro" />
-    </xacro:unless>
-    <xacro:if value="$(arg use_ros2_control)">
-        <xacro:include filename="ros2_control.xacro" />
+<robot xmlns:xacro="http://ros.org/wiki/xacro" name="$(arg robot_name)">
+    <xacro:include filename="$(find description)/urdf/inertia_macro.urdf.xacro"/>
+    <xacro:include filename="$(find description)/urdf/minibot.urdf.xacro"/>
+    <xacro:include filename="$(find description)/urdf/minibot_gazebo.urdf.xacro"/>
+    <xacro:include filename="$(find description)/urdf/minibot_ros2_control.urdf.xacro"/>
+    <xacro:arg name="prefix" default=""/>
+    <xacro:arg name="is_sim" default="false"/>
+    <xacro:arg name="robot_port_name" default="/dev/ttyArduino"/>
+    <xacro:arg name="robot_baudrate" default="500000"/>
+    <xacro:property name="prefix" value="$(arg prefix)"/>
+    <!-- insert robot base -->
+    <xacro:insert_robot prefix="$(arg prefix)"/>
+    <xacro:insert_ros2_control prefix="$(arg prefix)" is_sim="$(arg is_sim)" robot_port_name="$(arg robot_port_name)" robot_baudrate="$(arg robot_baudrate)"/>
+    <xacro:if value="$(arg is_sim)">
+        <xacro:insert_gazebo prefix="$(arg prefix)"/>
     </xacro:if>
-    <xacro:include filename="lidar.xacro" />
-    <xacro:include filename="camera.xacro" />
+    <!-- insert ydlidar_x2 lidar -->
+    <link name="${prefix}ydlidar_lidar_mount">
+        <visual>
+            <origin xyz="0 0 0" rpy="0 0 0"/>
+            <geometry>
+                <mesh filename="package://description/meshes/visual/ydlidar_x2_assy.dae" scale="1 1 1"/>
+            </geometry>
+        </visual>
+        <collision>
+            <origin xyz="0 0 0" rpy="0 0 0"/>
+            <geometry>
+                <mesh filename="package://description/meshes/collision/ydlidar_x2_assy.stl" scale="1 1 1"/>
+            </geometry>
+        </collision>
+        <inertial>
+            <origin xyz="0.007 0 0.025" rpy="0 0 0"/>
+            <mass value="0.150"/>
+            <inertia ixx="0.000058" ixy="0" ixz="0.000005" iyy="0.000099" iyz="0" izz="0.000103"/>
+        </inertial>
+    </link>
+    <joint name="${prefix}idar_mount_fixed_joint" type="fixed">
+        <parent link="${prefix}base_link"/>
+        <child link="${prefix}ydlidar_lidar_mount"/>
+        <origin xyz="-0.01 0 0.085" rpy="0 0 0"/>
+    </joint>
+    <link name="${prefix}laser_link"/>
+    <joint name="${prefix}laser_link_fixed_joint" type="fixed">
+        <parent link="${prefix}ydlidar_lidar_mount"/>
+        <child link="${prefix}laser_link"/>
+        <origin xyz="0 0 0.04245" rpy="0 0 0"/>
+    </joint>
 </robot>
